File: PCB_Draft_2/PCB_Draft_2.brd (EAGLE design)
At the start: 76.2 x 50.8 mm, 19 parts

Commit message: MD Screwterm labels & optimizations
Parts:
- added JP1, JP2: (no value), jumper:JP1
- added SW1, SW2: PUSHBUTTON, ME507:B3F-10XX
- moved D 34.2 mm to (15.2, 35.6), turned to 180 degrees
- moved D_CH 31.4 mm to (3.81, 34.3), turned to 90 degrees
- moved C1 20.7 mm to (24.1, 35.6)
- moved C2 20.7 mm to (24.1, 31.8)
- moved R3 20.7 mm to (24.1, 27.9)
- moved I2C 18.2 mm to (7.62, 48.3), turned to 180 degrees
- moved A 8.13 mm to (34.3, 35.6)
- moved A_CH 5.68 mm to (34.3, 47.0)
- moved A_COM 3.59 mm to (19.1, 47.0), turned to 180 degrees
Connections:
- new net ENC_A: X1.5
- new net ENC_B: X1.8
- net 3.3V: now also X1.9
- net GND: now also X1.10
Routing:
- net 9V: track 53.7 -> 58.7 mm
Other:
- board text added: "+"
- board text added: "-"
- board text added: "Aux Enc"
- board text added: "E"
- board text added: "Motor A"
- board text added: "Motor B"
- board text added: "Motor Power In"

Commit message: Near-final draft - all wires run; checking formatting
Parts:
- removed R1, R2: 4.7k, rcl:M0805
- added PU_SCL, PU_SDA: 4.7k, rcl:M0805
- added SD_READ: (no value), con-lsta:FE08
- D_CH: device ME507:8POL254 -> ME507:6POL254
- I2C: device con-lstb:MA04-1 -> ME507:4POL254
- moved A_CH 46.8 mm to (3.81, 11.4), turned to 90 degrees
- moved SW1 42.4 mm to (38.1, 44.3)
- moved SW2 39.7 mm to (16.4, 44.5), turned to 270 degrees
- moved JP1 35.9 mm to (40.4, 37.1), turned to 90 degrees
- moved A 31.5 mm to (14.0, 11.4), turned to 270 degrees
- moved JP2 31.4 mm to (14.2, 37.5), turned to 90 degrees
- moved C2 26.0 mm to (16.5, 6.86), turned to 180 degrees
- moved A_COM 25.4 mm to (3.81, 26.7), turned to 270 degrees
- moved C1 21.2 mm to (16.5, 15.7), turned to 180 degrees
- moved I2C 20.1 mm to (27.3, 44.5), turned to 0 degrees
- moved R3 12.0 mm to (12.7, 24.1)
- moved D_CH 7.62 mm to (3.81, 41.9)
- moved D 4.02 mm to (14.0, 31.8), turned to 270 degrees
- renumbered MD_2 to MD
Connections:
- new net N$24: FTHRWNG.11, SD_READ.4
- new net N$26: JP1.1, SW1.3, SW1.4
- new net N$27: JP2.2, SW2.3, SW2.4
- new net N$28: FTHRWNG.13, SD_READ.5
- new net N$29: FTHRWNG.8, JP2.1
- new net N$30: FTHRWNG.7, JP1.2
- new net N$31: FTHRWNG.12, SD_READ.6
- net 3.3V: now also PU_SCL.1, PU_SDA.1, SD_READ.2, SW1.1, SW1.2, SW2.1, SW2.2; no longer R1.1, R2.1
- net ENC_A: now also FTHRWNG.9
- net ENC_B: now also FTHRWNG.10
- net GND: now also SD_READ.3
- net N$1: no longer D_CH.1
- net N$2: no longer D_CH.2
- net N$3: now also D_CH.1; no longer D_CH.3
- net N$4: now also D_CH.2; no longer D_CH.4
- net N$5: now also D_CH.3; no longer D_CH.5
- net N$6: now also D_CH.4; no longer D_CH.6
- net N$7: now also D_CH.5; no longer D_CH.7
- net N$8: now also D_CH.6; no longer D_CH.8
- net SCL: now also PU_SCL.2; no longer R2.2
- net SDA: now also PU_SDA.2; no longer R1.2
Routing:
- net 3.3V: track 0.00 -> 178.8 mm, vias 0 -> 4
- net SCL: track 0.00 -> 90.8 mm, vias 0 -> 4
- net SDA: track 0.00 -> 85.5 mm, vias 0 -> 6
- net N$29: track 0.00 -> 54.6 mm, vias 0 -> 4
- net N$30: track 0.00 -> 51.5 mm, vias 0 -> 2
- net N$19: track 0.00 -> 47.8 mm, vias 0 -> 2
- net ENC_A: track 0.00 -> 44.0 mm, vias 0 -> 2
- net ENC_B: track 0.00 -> 35.4 mm, vias 0 -> 2
- net COM: track 0.00 -> 28.1 mm, vias 0 -> 2
- net N$8: track 0.00 -> 22.1 mm
- net N$3: track 0.00 -> 22.0 mm
- net N$4: track 0.00 -> 22.0 mm
- net N$7: track 0.00 -> 19.9 mm
- net N$6: track 0.00 -> 17.7 mm
- net N$5: track 0.00 -> 15.3 mm
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Other:
- board text added: "Encoder Power Out"
- board text removed: "Aux Enc"
