File: PCB_Draft_2/PCB_Draft_2.sch (EAGLE design)
At the start: 19 parts

Commit message: MD Screwterm labels & optimizations
Parts:
- added JP1, JP2: (no value), jumper:JP1E
- added SW1, SW2: PUSHBUTTON, ME507:PUSHBUTTON
Connections:
- new net ENC_A: X1-5.1
- new net ENC_B: X1-8.1
- net 3.3V: now also X1-9.1
- net GND: now also X1-10.1
Changed lines of the file:
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@@
 <part name="R5" library="rcl" library_urn="urn:adsk.eagle:library:334" deviceset="R-US_" device="M0805" package3d_urn="urn:adsk.eagle:package:23556/2" value="100"/>
 <part name="X1" library="ME507" deviceset="SCREWTERM_10P" device="_254"/>
+<part name="SW1" library="ME507" deviceset="PUSHBUTTON" device="" package3d_urn="urn:adsk.eagle:package:27496/1"/>
+<part name="SW2" library="ME507" deviceset="PUSHBUTTON" device="" package3d_urn="urn:adsk.eagle:package:27496/1"/>
+<part name="JP1" library="jumper" library_urn="urn:adsk.eagle:library:252" deviceset="JP1E" device="" package3d_urn="urn:adsk.eagle:package:15455/1"/>
+<part name="JP2" library="jumper" library_urn="urn:adsk.eagle:library:252" deviceset="JP1E" device="" package3d_urn="urn:adsk.eagle:package:15455/1"/>
 </parts>
 <sheets>
@@
 <attribute name="VALUE" x="359.664" y="161.798" size="1.778" layer="96"/>
 </instance>
+<instance part="SW1" gate="1" x="121.92" y="198.12" smashed="yes">
+<attribute name="NAME" x="119.38" y="204.47" size="1.778" layer="95"/>
+<attribute name="VALUE" x="125.095" y="201.93" size="1.778" layer="96"/>
+</instance>
+<instance part="SW2" gate="1" x="121.92" y="182.88" smashed="yes">
+<attribute name="NAME" x="119.38" y="189.23" size="1.778" layer="95"/>
+<attribute name="VALUE" x="125.095" y="186.69" size="1.778" layer="96"/>
+</instance>
+<instance part="JP1" gate="A" x="101.6" y="198.12" smashed="yes">
+<attribute name="NAME" x="100.33" y="198.12" size="1.778" layer="95" rot="R90"/>
+<attribute name="VALUE" x="107.315" y="198.12" size="1.778" layer="96" rot="R90"/>
+</instance>
+<instance part="JP2" gate="A" x="101.6" y="182.88" smashed="yes">
+<attribute name="NAME" x="100.33" y="182.88" size="1.778" layer="95" rot="R90"/>
+<attribute name="VALUE" x="107.315" y="182.88" size="1.778" layer="96" rot="R90"/>
+</instance>
 </instances>
 <busses>
@@
 <wire x1="177.8" y1="200.66" x2="170.18" y2="200.66" width="0.1524" layer="91"/>
 <label x="170.18" y="200.66" size="1.778" layer="95"/>
+</segment>
+<segment>
+<pinref part="X1" gate="-10" pin="1"/>
+<wire x1="358.14" y1="165.1" x2="347.98" y2="165.1" width="0.1524" layer="91"/>
+<label x="347.98" y="165.1" size="1.778" layer="95"/>
 </segment>
 </net>
@@
 <label x="170.18" y="205.74" size="1.778" layer="95"/>
 </segment>
+<segment>
+<pinref part="X1" gate="-9" pin="1"/>
+<wire x1="358.14" y1="170.18" x2="347.98" y2="170.18" width="0.1524" layer="91"/>
+<label x="347.98" y="170.18" size="1.778" layer="95"/>
+</segment>
 </net>
 <net name="N$1" class="0">
@@
 </segment>
 </net>
+<net name="ENC_A" class="0">
+<segment>
+<pinref part="X1" gate="-5" pin="1"/>
+<wire x1="358.14" y1="190.5" x2="337.82" y2="190.5" width="0.1524" layer="91"/>
+<label x="337.82" y="190.5" size="1.778" layer="95"/>
+</segment>
+</net>
+<net name="ENC_B" class="0">
+<segment>
+<pinref part="X1" gate="-8" pin="1"/>
+<wire x1="358.14" y1="175.26" x2="337.82" y2="175.26" width="0.1524" layer="91"/>
+<label x="337.82" y="175.26" size="1.778" layer="95"/>
+</segment>
+</net>

Commit message: Near-final draft - all wires run; checking formatting
Parts:
- removed MD_2: L6205D, st-microelectronics:L6205D
- removed R1, R2: 4.7k, rcl:R-US_M0805
- added MD: L6205D, st-microelectronics:L6205D
- added PU_SCL, PU_SDA: 4.7k, rcl:R-US_M0805
- added SD_READ: (no value), con-lsta:FE08-1
- D_CH: device ME507:SCREWTERM_8P_254 -> ME507:SCREWTERM_6P_254
- I2C: device con-lstb:MA04-1 -> ME507:SCREWTERM_4P_254
Connections:
- new net N$24: FTHRWNG.GPIOSCK, SD_READ.4
- new net N$26: JP1.1, SW1.P, SW1.P1
- new net N$27: JP2.2, SW2.P, SW2.P1
- new net N$28: FTHRWNG.GPIOMISO, SD_READ.5
- new net N$29: FTHRWNG.GPIOA3, JP2.1
- new net N$30: FTHRWNG.GPIOA2, JP1.2
- new net N$31: FTHRWNG.GPIOMOSI, SD_READ.6
- net 3.3V: now also I2C-1.1, PU_SCL.1, PU_SDA.1, SD_READ.2, SW1.S, SW1.S1, SW2.S, SW2.S1; no longer I2C.1, R1.1, R2.1
- net 9V: now also MD.VS_A, MD.VS_B; no longer MD_2.VS_A, MD_2.VS_B
- net ENC_A: now also FTHRWNG.GPIOA4
- net ENC_B: now also FTHRWNG.GPIOA5
- net GND: now also I2C-4.1, MD.GND, MD.GND@1, MD.GND@2, MD.GND@3, SD_READ.3; no longer I2C.4, MD_2.GND, MD_2.GND@1, MD_2.GND@2, MD_2.GND@3
- net M1A: now also MD.OUT1A; no longer MD_2.OUT1A
- net M1B: now also MD.OUT1B; no longer MD_2.OUT1B
- net M2A: now also MD.OUT2A; no longer MD_2.OUT2A
- net M2B: now also MD.OUT2B; no longer MD_2.OUT2B
- net MGND: now also MD.SENSE_A, MD.SENSE_B; no longer MD_2.SENSE_A, MD_2.SENSE_B
- net N$1: no longer D_CH-1.1
- net N$18: now also MD.EN_B; no longer MD_2.EN_B
- net N$2: no longer D_CH-2.1
- net N$20: now also MD.IN2_B; no longer MD_2.IN2_B
- net N$21: now also MD.IN1_B; no longer MD_2.IN1_B
- net N$22: now also MD.IN2_A; no longer MD_2.IN2_A
- net N$23: now also MD.IN1_A; no longer MD_2.IN1_A
- net N$25: now also MD.EN_A; no longer MD_2.EN_A
- net N$3: now also D_CH-1.1; no longer D_CH-3.1
- net N$4: now also D_CH-2.1; no longer D_CH-4.1
- net N$43: now also MD.VCP; no longer MD_2.VCP
- net N$46: now also MD.VBOOT; no longer MD_2.VBOOT
- net N$5: now also D_CH-3.1; no longer D_CH-5.1
- net N$6: now also D_CH-4.1; no longer D_CH-6.1
- net N$7: now also D_CH-5.1; no longer D_CH-7.1
- net N$8: now also D_CH-6.1; no longer D_CH-8.1
- net SCL: now also I2C-3.1, PU_SCL.2; no longer I2C.3, R2.2
- net SDA: now also I2C-2.1, PU_SDA.2; no longer I2C.2, R1.2
Other:
- moved on the sheet: A, A_CH-1, A_CH-2, A_CH-3, A_CH-4, A_CH-5, A_CH-6, A_CH-7, A_CH-8, A_COM-1, A_COM-2, A_COM-3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
