File: PCB_Draft_3/PCB_Draft_3.brd (EAGLE design)
At the start: 76.2 x 50.8 mm, 24 parts, among them SW1 PUSHBUTTON, SW2 PUSHBUTTON

Commit message: Near-final draft - all wires run; checking formatting
Parts:
- removed A: ADS7828, burr-brown:TSSOP16-PW
- removed A_COM: (no value), ME507:3POL254
- removed C1, C2: (no value), rcl:C0805
- removed D: PCA9534PW, micro-philips:TSSOP16
- removed D_CH: (no value), ME507:6POL254
- added D_A: (no value), ME507:8POL254
- added D_EXP_A, D_EXP_B: PCA9534PW, micro-philips:TSSOP16
- added LED1, LED2: (no value), led:CHIPLED_0805
- added PU_SCL, PU_SDA: 4.7k, rcl:M0805
- added P_OUT: (no value), ME507:2POL254
- R1, R2: value 4.7k -> (none)
- R3: value 0 -> 10k
- moved R1 58.2 mm to (12.7, 47.0)
- moved R2 39.9 mm to (41.9, 47.0), turned to 0 degrees
- moved R3 18.9 mm to (19.1, 6.35), turned to 270 degrees
- moved JP1 5.73 mm to (32.8, 35.8), turned to 180 degrees
- moved SW1 4.58 mm to (38.1, 40.5)
- moved SW2 3.81 mm to (16.4, 40.6)
- moved JP2 3.14 mm to (21.1, 35.3), turned to 180 degrees
- moved I2C 1.91 mm to (27.3, 44.5)
- renumbered A_CH to D_B
Connections:
- removed net COM: A.11, A_COM.3, R3.1
- removed net ENC_A: FTHRWNG.9, X1.5
- removed net ENC_B: FTHRWNG.10, X1.8
- removed net N$30: FTHRWNG.7, JP1.2
- new net CD: FTHRWNG.9, SD_READ.8
- new net CLK: FTHRWNG.11, SD_READ.4
- new net CS: FTHRWNG.10, SD_READ.7
- new net DI: FTHRWNG.12, SD_READ.6
- new net DO: FTHRWNG.13, SD_READ.5
- new net ENC1_A: FTHRWNG.5, X1.5
- new net ENC1_B: FTHRWNG.6, X1.9
- new net ENC2_A: FTHRWNG.7, X1.6
- new net ENC2_B: FTHRWNG.8, X1.10
- new net N$24: JP2.2, LED1.A, SW2.1, SW2.2
- new net N$28: LED1.C, R1.1
- net 3.3V: now also D_EXP_A.16, D_EXP_B.16, JP1.1, JP2.1, PU_SCL.1, PU_SDA.1, P_OUT.1, R3.2, SD_READ.2; no longer A.16, A_COM.1, C1.1, D.16, R1.1, R2.1, SW1.1, SW1.2, SW2.1, SW2.2, X1.9
- net GND: now also D_EXP_A.1, D_EXP_A.2, D_EXP_A.3, D_EXP_A.8, D_EXP_B.1, D_EXP_B.2, D_EXP_B.8, P_OUT.2, R1.2, R2.2, SD_READ.3; no longer A.12, A.13, A.9, A_COM.2, C1.2, C2.2, D.1, D.2, D.3, D.8, R3.2, X1.10
- net M1B: now also X1.7; no longer X1.6
- net M2B: now also X1.8; no longer X1.7
- net N$1: now also D_A.1, D_EXP_A.12, SW2.3, SW2.4; no longer D.12
- net N$10: now also D_EXP_B.5; no longer A.2
- net N$11: now also D_EXP_B.6; no longer A.3
- net N$12: now also D_EXP_B.7; no longer A.4
- net N$13: now also D_EXP_B.9; no longer A.5
- net N$14: now also D_EXP_B.10; no longer A.6
- net N$15: now also D_EXP_B.11; no longer A.7
- net N$16: now also D_EXP_B.12; no longer A.8
- net N$17: now also LED2.C, R2.1; no longer A.10, C2.1
- net N$19: now also D_EXP_A.13; no longer D.13
- net N$2: now also D_A.2, D_EXP_A.11, SW1.3, SW1.4; no longer D.11
- net N$26: now also JP1.2, LED2.A, SW1.1, SW1.2; no longer JP1.1, SW1.3, SW1.4
- net N$27: now also D_EXP_B.13, FTHRWNG.16; no longer JP2.2, SW2.3, SW2.4
- net N$29: now also D_EXP_B.3, R3.1; no longer FTHRWNG.8, JP2.1
- net N$3: now also D_A.3, D_EXP_A.10; no longer D.10, D_CH.1
- net N$4: now also D_A.4, D_EXP_A.9; no longer D.9, D_CH.2
- net N$5: now also D_A.5, D_EXP_A.7; no longer D.7, D_CH.3
- net N$6: now also D_A.6, D_EXP_A.6; no longer D.6, D_CH.4
- net N$7: now also D_A.7, D_EXP_A.5; no longer D.5, D_CH.5
- net N$8: now also D_A.8, D_EXP_A.4; no longer D.4, D_CH.6
- net N$9: now also D_EXP_B.4; no longer A.1
- net SCL: now also D_EXP_A.14, D_EXP_B.14, PU_SCL.2; no longer A.14, D.14, R2.2
- net SDA: now also D_EXP_A.15, D_EXP_B.15, PU_SDA.2; no longer A.15, D.15, R1.2
Routing:
- net 3.3V: track 178.8 -> 115.3 mm
- net M2B: track 53.6 -> 0.00 mm, vias 4 -> 0
- net N$29: track 52.8 -> 0.00 mm, vias 4 -> 0
- net N$30: track 48.8 -> 0.00 mm, vias 2 -> 0
- net ENC_A: track 43.5 -> 0.00 mm, vias 2 -> 0
- net ENC_B: track 34.9 -> 0.00 mm, vias 2 -> 0
- net M1B: track 33.9 -> 0.00 mm, vias 2 -> 0
- net COM: track 28.1 -> 0.00 mm, vias 2 -> 0
- net SCL: track 94.5 -> 77.6 mm, vias 4 -> 2
- net N$3: track 22.0 -> 6.41 mm
- net N$24: track 0.00 -> 15.1 mm
- net SDA: track 88.7 -> 73.8 mm, vias 6 -> 4
- net N$4: track 22.0 -> 8.76 mm
- net N$19: track 47.8 -> 34.7 mm, vias 2 -> 0
- net N$27: track 11.6 -> 0.00 mm
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Other:
- board text added: "E1_A"
- board text added: "E1_B"
- board text added: "E2_A"
- board text added: "E2_B"
- board text removed: "E"
- board text removed: "Encoder Power Out"
