File: PCB_Draft_4/PCB_Draft_4.brd (EAGLE design)
At the start: 76.2 x 50.8 mm, 24 parts, among them SW1 PUSHBUTTON, SW2 PUSHBUTTON

Commit message: Near-final draft - all wires run; checking formatting
Parts:
- removed A_CH: (no value), ME507:8POL254
- removed D: PCA9534PW, micro-philips:TSSOP16
- removed D_CH: (no value), ME507:6POL254
- removed JP1, JP2: (no value), jumper:JP1
- removed R1, R2: 4.7k, rcl:M0805
- removed R3: 0, rcl:M0805
- removed SW1, SW2: PUSHBUTTON, ME507:B3F-10XX
- removed X1: (no value), ME507:10POL254
- added A_TERM: (no value), ME507:6POL254
- added D_I2C: PCA9534PW, micro-philips:TSSOP16
- added D_TERM: (no value), ME507:8POL254
- added JP1_A, JP1_B, JP2_A, JP2_B: (no value), jumper:JP1
- added LED1, LED2: (no value), led:CHIP-LED0805
- added M_TERM: (no value), ME507:12POL254
- added PU_SCL, PU_SDA, R_L1, R_L2: 4.7k, rcl:M0805
- added R_COM: 0, rcl:M0805
- added USER_1, USER_2: PUSHBUTTON, ME507:B3F-10XX
- moved A_COM 5.08 mm to (3.81, 21.6)
- moved I2C 1.57 mm to (27.7, 44.1)
- moved C1 1.20 mm to (17.1, 16.8)
- moved C2 0.76 mm to (16.5, 6.10)
- renumbered A to A_I2C, C5 to C_M1, C6 to C_M2, D3 to D_M1, D4 to D_M2, R5 to R_M
Connections:
- net N$43 renamed VCP
- net N$46 renamed VBOOT
- removed net 3.3V: A_COM.1, A_I2C.16, C1.1, D.16, FTHRWNG.2, I2C.1, R1.1, R2.1, SW1.1, SW1.2, SW2.1, SW2.2, X1.9
- removed net 9V: C_M1.1, D_M1.A, MD.14, MD.17, X1.1
- removed net ENC_A: FTHRWNG.9, X1.5
- removed net ENC_B: FTHRWNG.10, X1.8
- removed net MGND: MD.3, MD.8, X1.2
- removed net N$15: A_CH.2, A_I2C.7
- removed net N$16: A_CH.1, A_I2C.8
- removed net N$7: D.5, D_CH.5
- new net CD: FTHRWNG.9, SD_READ.8
- new net CLK: FTHRWNG.11, SD_READ.4
- new net CS: FTHRWNG.10, SD_READ.7
- new net DI: FTHRWNG.12, SD_READ.6
- new net DO: FTHRWNG.13, SD_READ.5
- new net ENC1_A: FTHRWNG.5, M_TERM.5
- new net ENC1_B: FTHRWNG.7, M_TERM.9
- new net ENC2_A: FTHRWNG.6, M_TERM.6
- new net ENC2_B: FTHRWNG.8, M_TERM.10
- new net GND_MOT: MD.3, MD.8, M_TERM.2
- new net N$32: D_I2C.5, D_TERM.5
- new net N$33: D_I2C.4, D_TERM.6
- new net N$35: D_TERM.8, JP2_B.1
- new net V_LOG: A_COM.1, A_I2C.16, C1.1, D_I2C.16, FTHRWNG.2, I2C.1, JP1_A.1, JP2_A.2, M_TERM.11, PU_SCL.1, PU_SDA.1, SD_READ.2
- new net V_MOT: C_M1.1, D_M1.A, MD.14, MD.17, M_TERM.1
- net COM: now also R_COM.1; no longer R3.1
- net GND: now also D_I2C.1, D_I2C.2, D_I2C.3, D_I2C.8, M_TERM.12, R_COM.2, R_L1.2, R_L2.1, SD_READ.3; no longer D.1, D.2, D.3, D.8, R3.2, X1.10
- net M1A: now also M_TERM.3; no longer X1.3
- net M1B: now also M_TERM.7; no longer X1.6
- net M2A: now also M_TERM.4; no longer X1.4
- net M2B: now also M_TERM.8; no longer X1.7
- net N$1: now also D_I2C.12, JP2_B.2, USER_2.1, USER_2.2; no longer D.12
- net N$10: now also A_TERM.5; no longer A_CH.7
- net N$11: now also A_TERM.4; no longer A_CH.6
- net N$12: now also A_TERM.3; no longer A_CH.5
- net N$13: now also A_TERM.2; no longer A_CH.4
- net N$14: now also A_TERM.1; no longer A_CH.3
- net N$19: now also D_I2C.13; no longer D.13
- net N$2: now also D_I2C.11, JP1_B.1, USER_1.1, USER_1.2; no longer D.11
- net N$26: now also JP1_A.2, LED1.A, USER_1.3, USER_1.4; no longer JP1.1, SW1.3, SW1.4
- net N$27: now also JP2_A.1, LED2.A, USER_2.3, USER_2.4; no longer JP2.2, SW2.3, SW2.4
- net N$29: now also LED1.C, R_L1.1; no longer FTHRWNG.8, JP2.1
- net N$3: now also D_I2C.10, D_TERM.1; no longer D.10, D_CH.1
- net N$30: now also LED2.C, R_L2.2; no longer FTHRWNG.7, JP1.2
- net N$4: now also D_I2C.9, D_TERM.2; no longer D.9, D_CH.2
- net N$5: now also D_I2C.7, D_TERM.3; no longer D.7, D_CH.3
- net N$6: now also D_I2C.6, D_TERM.4; no longer D.6, D_CH.4
- net N$8: now also D_TERM.7, JP1_B.2; no longer D.4, D_CH.6
- net N$9: now also A_TERM.6; no longer A_CH.8
- net SCL: now also D_I2C.14, PU_SCL.2; no longer D.14, R2.2
- net SDA: now also D_I2C.15, PU_SDA.2; no longer D.15, R1.2
Routing:
- net 3.3V: track 178.8 -> 0.00 mm, vias 4 -> 0
- net V_LOG: track 0.00 -> 160.5 mm, vias 0 -> 4
- net ENC1_A: track 0.00 -> 60.3 mm, vias 0 -> 2
- net 9V: track 58.7 -> 0.00 mm
- net ENC2_A: track 0.00 -> 58.3 mm, vias 0 -> 2
- net V_MOT: track 0.00 -> 53.8 mm
- net N$29: track 52.8 -> 8.56 mm, vias 4 -> 0
- net ENC_A: track 43.5 -> 0.00 mm, vias 2 -> 0
- net ENC1_B: track 0.00 -> 42.5 mm, vias 0 -> 4
- net N$30: track 48.8 -> 8.46 mm, vias 2 -> 0
- net ENC2_B: track 0.00 -> 40.0 mm, vias 0 -> 4
- net N$1: track 0.00 -> 37.9 mm, vias 0 -> 2
- net ENC_B: track 34.9 -> 0.00 mm, vias 2 -> 0
- net N$35: track 0.00 -> 32.7 mm
- net N$2: track 0.00 -> 22.6 mm, vias 0 -> 1
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- added copper zone on layer 1, net GND_MOT
- added copper zone on layer 16, net GND_MOT
- added copper zone on layer 1, net V_MOT
- removed copper zone on layer 1, net 9V
- removed copper zone on layer 1, net MGND
- removed copper zone on layer 16, net MGND
Other:
- board text added: "1"
- board text added: "2"
- board text added: "3"
- board text added: "3.3V"
- board text added: "4"
- board text added: "5"
- board text added: "6"
- board text added: "ANALOG_I2C"
- board text added: "COM"
- board text added: "ENC_1"
- board text added: "ENC_2"
- board text added: "GND"
- board text added: "GPIO_I2C"
- board text added: "SCL"
- board text added: "SDA"
- board text added: "U1/7"
- board text added: "U2/8"
- board text added: "V_M IN"
- board text removed: "E"
- board text removed: "Encoder Power Out"
- board text removed: "Motor Power In"

Commit message: Final-ish Version - for review
Parts:
- C1: value (none) -> 1u
- C2: value (none) -> 0.1u
- moved R_COM 1.27 mm to (11.9, 20.4)
- moved PU_SCL 0.13 mm to (61.0, 12.7)
Connections:
- net N$19 renamed INT
- net V_LOG renamed +3V3
Routing:
- net +3V3: track 160.5 -> 155.7 mm
- net SCL: track 90.4 -> 93.5 mm
- net COM: track 26.0 -> 23.6 mm
- net N$18: track 32.3 -> 33.3 mm
- net N$25: track 29.7 -> 30.3 mm
- net GND: track 23.7 -> 23.1 mm
- added copper zone on layer 1, net +3V3
