File: PCB_Draft_4/PCB_Draft_4.sch (EAGLE design)
At the start: 24 parts, among them SW1 PUSHBUTTON, SW2 PUSHBUTTON

Commit message: Near-final draft - all wires run; checking formatting
Parts:
- removed A: ADS7828, burr-brown:ADS7828
- removed A_CH: (no value), ME507:SCREWTERM_8P_254
- removed C5: 220n, rcl:C-USC0805
- removed C6: 10n, rcl:C-USC0805
- removed D: PCA9534PW, micro-philips:PCA9534PW
- removed D3, D4: 1N4148DO35-7, diode:1N4148DO35-7
- removed D_CH: (no value), ME507:SCREWTERM_6P_254
- removed JP1, JP2: (no value), jumper:JP1E
- removed R1, R2: 4.7k, rcl:R-US_M0805
- removed R3: 0, rcl:R-US_M0805
- removed R5: 100, rcl:R-US_M0805
- removed SV1: (no value), con-lsta:FE08-1
- removed SW1, SW2: PUSHBUTTON, ME507:PUSHBUTTON
- removed X1: (no value), ME507:SCREWTERM_10P_254
- added A_I2C: ADS7828, burr-brown:ADS7828
- added A_TERM: (no value), ME507:SCREWTERM_6P_254
- added C_M1: 220n, rcl:C-USC0805
- added C_M2: 10n, rcl:C-USC0805
- added D_I2C: PCA9534PW, micro-philips:PCA9534PW
- added D_M1, D_M2: 1N4148DO35-7, diode:1N4148DO35-7
- added D_TERM: (no value), ME507:SCREWTERM_8P_254
- added JP1_A, JP1_B, JP2_A, JP2_B: (no value), jumper:JP1E
- added LED1, LED2: (no value), led:LEDCHIP-LED0805
- added M_TERM: (no value), ME507:SCREWTERM_12P_254
- added PU_SCL, PU_SDA, R_L1, R_L2: 4.7k, rcl:R-US_M0805
- added R_COM: 0, rcl:R-US_M0805
- added R_M: 100, rcl:R-US_M0805
- added SD_READ: (no value), con-lsta:FE08-1
- added USER_1, USER_2: PUSHBUTTON, ME507:PUSHBUTTON
Connections:
- removed net 3.3V: A.VDD, A_COM-1.1, C1.1, D.VDD, FTHRWNG.3V, I2C-1.1, R1.1, R2.1, SW1.S, SW1.S1, SW2.S, SW2.S1, X1-9.1
- removed net 9V: C5.1, D3.A, MD.VS_A, MD.VS_B, X1-1.1
- removed net ENC_A: FTHRWNG.GPIOA4, X1-5.1
- removed net ENC_B: FTHRWNG.GPIOA5, X1-8.1
- removed net MGND: MD.SENSE_A, MD.SENSE_B, X1-2.1
- removed net N$15: A.CH6, A_CH-2.1
- removed net N$16: A.CH7, A_CH-1.1
- removed net N$43: C6.2, MD.VCP
- removed net N$46: C5.2, D4.C, MD.VBOOT
- removed net N$7: D.IO1, D_CH-5.1
- new net CD: FTHRWNG.GPIOA4, SD_READ.8
- new net CLK: FTHRWNG.GPIOSCK, SD_READ.4
- new net CS: FTHRWNG.GPIOA5, SD_READ.7
- new net DI: FTHRWNG.GPIOMOSI, SD_READ.6
- new net DO: FTHRWNG.GPIOMISO, SD_READ.5
- new net ENC1_A: FTHRWNG.GPIOA0, M_TERM-5.1
- new net ENC1_B: FTHRWNG.GPIOA2, M_TERM-9.1
- new net ENC2_A: FTHRWNG.GPIOA1, M_TERM-6.1
- new net ENC2_B: FTHRWNG.GPIOA3, M_TERM-10.1
- new net GND_MOT: MD.SENSE_A, MD.SENSE_B, M_TERM-2.1
- new net N$32: D_I2C.IO1, D_TERM-5.1
- new net N$33: D_I2C.IO0, D_TERM-6.1
- new net N$35: D_TERM-8.1, JP2_B.1
- new net VBOOT: C_M1.2, D_M2.C, MD.VBOOT
- new net VCP: C_M2.2, MD.VCP
- new net V_LOG: A_COM-1.1, A_I2C.VDD, C1.1, D_I2C.VDD, FTHRWNG.3V, I2C-1.1, JP1_A.1, JP2_A.2, M_TERM-11.1, PU_SCL.1, PU_SDA.1, SD_READ.2
- new net V_MOT: C_M1.1, D_M1.A, MD.VS_A, MD.VS_B, M_TERM-1.1
- net COM: now also A_I2C.COM, R_COM.1; no longer A.COM, R3.1
- net GND: now also A_I2C.A0, A_I2C.A1, A_I2C.GND, D_I2C.A0, D_I2C.A1, D_I2C.A2, D_I2C.VSS, M_TERM-12.1, R_COM.2, R_L1.2, R_L2.1, SD_READ.3; no longer A.A0, A.A1, A.GND, D.A0, D.A1, D.A2, D.VSS, R3.2, X1-10.1
- net M1A: now also M_TERM-3.1; no longer X1-3.1
- net M1B: now also M_TERM-7.1; no longer X1-6.1
- net M2A: now also M_TERM-4.1; no longer X1-4.1
- net M2B: now also M_TERM-8.1; no longer X1-7.1
- net N$1: now also D_I2C.IO7, JP2_B.2, USER_2.S, USER_2.S1; no longer D.IO7
- net N$10: now also A_I2C.CH1, A_TERM-5.1; no longer A.CH1, A_CH-7.1
- net N$11: now also A_I2C.CH2, A_TERM-4.1; no longer A.CH2, A_CH-6.1
- net N$12: now also A_I2C.CH3, A_TERM-3.1; no longer A.CH3, A_CH-5.1
- net N$13: now also A_I2C.CH4, A_TERM-2.1; no longer A.CH4, A_CH-4.1
- net N$14: now also A_I2C.CH5, A_TERM-1.1; no longer A.CH5, A_CH-3.1
- net N$17: now also A_I2C.REFIN/REFOUT; no longer A.REFIN/REFOUT
- net N$19: now also D_I2C.!INT; no longer D.!INT
- net N$2: now also D_I2C.IO6, JP1_B.1, USER_1.S, USER_1.S1; no longer D.IO6
- net N$26: now also JP1_A.2, LED1.A, USER_1.P, USER_1.P1; no longer JP1.1, SW1.P, SW1.P1
- net N$27: now also JP2_A.1, LED2.A, USER_2.P, USER_2.P1; no longer JP2.2, SW2.P, SW2.P1
- net N$29: now also LED1.C, R_L1.1; no longer FTHRWNG.GPIOA3, JP2.1
- net N$3: now also D_I2C.IO5, D_TERM-1.1; no longer D.IO5, D_CH-1.1
- net N$30: now also LED2.C, R_L2.2; no longer FTHRWNG.GPIOA2, JP1.2
- net N$4: now also D_I2C.IO4, D_TERM-2.1; no longer D.IO4, D_CH-2.1
- net N$44: now also C_M2.1, R_M.1; no longer C6.1, R5.1
- net N$45: now also D_M1.C, D_M2.A, R_M.2; no longer D3.C, D4.A, R5.2
- net N$5: now also D_I2C.IO3, D_TERM-3.1; no longer D.IO3, D_CH-3.1
- net N$6: now also D_I2C.IO2, D_TERM-4.1; no longer D.IO2, D_CH-4.1
- net N$8: now also D_TERM-7.1, JP1_B.2; no longer D.IO0, D_CH-6.1
- net N$9: now also A_I2C.CH0, A_TERM-6.1; no longer A.CH0, A_CH-8.1
- net SCL: now also A_I2C.SCL, D_I2C.SCL, PU_SCL.2; no longer A.SCL, D.SCL, R2.2
- net SDA: now also A_I2C.SDA, D_I2C.SDA, PU_SDA.2; no longer A.SDA, D.SDA, R1.2
Other:
- note added: "NOTE: USER INPUTS 1 & 2 ARE ENABLED AND DISABLED BY SWITCHING THE CORRESPONDING JUMPER BETWEEN LOCATION A TO LOCATION B. THIS ALLOWS DEVICES TO REMAIN CONNECTED TO TERMINALS D_TERM-7 AND D_TERM-8 WHEN USER INPUTS ARE ENABLED. LED INDICATORS ARE USED TO VISUALLY REPRESENT INPUT ACTIVATION."
- note added: "NOTE: VBOOT CIRCUIT USED FROM L6205D MANUAL"
- moved on the sheet: A_COM-1, A_COM-2, A_COM-3, C1, C2, I2C-1, I2C-2, I2C-3, I2C-4, MD

Commit message: Final-ish Version - for review
Parts:
- C1: value (none) -> 1u
- C2: value (none) -> 0.1u
Connections:
- net N$19 renamed INT
- net V_LOG renamed +3V3
Other:
- note added: "Adafruit HUZZAH32 ESP32 Feather Microcontroller"
- note added: "Disconnectable User Input Buttons"
- note added: "Header for SD Card Slot"
- note added: "I2C Analog Input Expansion"
- note added: "I2C GPIO Expander"
- note added: "I2C Screw Terminal"
- note added: "Motor Driver"
- note added: "NOTE: 4.7 kOHM PULLUP RESISTORS ARE INCLUDED TO ENABLE I2C COMMUNICATIONS."
- note added: "NOTE: DUE TO UNCLEAR DOCUMENTATION, IT IS NOT KNOWN IF THE COM CHANNEL OF THE EXPANDER SHOULD BE CONNECTED TO GROUND. R_COM IS A 0 OHM RESISTOR TO BE ADDED ONLY IF NECESSARY."
- note added: "NOTE: FOR COMPLETE MOTOR IMPLEMENTATION, EACH MOTOR HAS A 4-SCREW SECTION OF THE TERMINAL - 2 MOTOR LEADS AND 2 ENCODER LEADS. TO FACILITATE THIS, MOTOR POWER INPUT TERMINALS ARE LOCATED AT THE TOP OF THE SCREW TERMIAL AND LOGIC VOLTAGE TERMINALS ARE LOCATED AT THE BOTTOM OF THE TERMINAL."
- note added: "NOTE: HEADER CORRESPONDS TO ADAFRUIT MicroSD card breakout board+"
- moved on the sheet: C1, I2C-1, I2C-2, I2C-3, I2C-4, PU_SCL, PU_SDA, SD_READ, USER_1, USER_2
